Commit message: Nav2 rotation shim + lidar_yaw arg + base-driver passthrough
Physical Nav2 test on qb3rt-7 surfaced a chain of issues, all now fixed:

- RotationShimController wraps RPP (Jazzy replacement for the deprecated
  use_rotate_to_heading): pivots to face the path before driving and
  rotates to goal heading — the skid-steer "3-point turn". Verified live:
  NavigateToPose now pivots, drives, and settles without the fwd/back
  final-approach hunting. Surface-dependent: spins fine on vinyl, barely
  turns on carpet — noted in comments.
- Goal tolerances relaxed (xy 0.20->0.30, yaw 0.40->0.60): open-loop
  dead-reckoning odometry drifts vs AMCL.
- Velocity smoother angular cap 1.2->1.5 rad/s for shim pivot authority.
- lidar_yaw xacro arg + launch passthrough: scan-zero faces the chassis
  REAR on qb3rt-7 (verified by probing a nose-contact obstacle — raw scan
  ~180 deg), so pi remains correct there. The old lab map was mirrored
  because it was built while the drive was inverted (drive_inverted fix,
  0e357e8), NOT because the scan was flipped. Fresh map saved as lab2.
- odometry.launch.py forwards enable_base_driver to the base include so
  standalone bring-up gets the wheel driver.

Generated with [Devin](https://devin.ai)

Co-Authored-By: Devin <158243242+devin-ai-integration[bot]@users.noreply.github.com>

File: urdf/QB3rt.urdf.xacro (robot description, xacro)
@@ -1,4 +1,10 @@
 <?xml version="1.0"?>
 <robot xmlns:xacro="http://www.ros.org/wiki/xacro" name="teaching_QB3rt">
+  <!-- lidar_yaw: yaw from base_link +X to the lidar scan-zero. pi = scan-zero
+       faces the chassis REAR, so the +pi joint maps physical-front obstacles
+       to base +X. Verified on qb3rt-7 2026-07-19: a door touching the nose
+       read at raw scan ~180 deg -> zero faces rear -> lidar_yaw must be pi.
+       See the laser_joint comment for the full story. -->
+  <xacro:arg name="lidar_yaw" default="3.141592653589793"/>
   <!-- Dimensions are based on the provided drawing (mm -> m), with simple approximations. -->
   <xacro:property name="chassis_length" value="0.180"/>
@@ -101,17 +107,14 @@
     <parent link="base_link"/>
     <child link="laser_frame"/>
-    <!-- RPLIDAR C1 is physically mounted with its zero-angle reference facing
-         the chassis REAR, not the front as originally assumed here. Confirmed
-         2026-07-13: with Fixed Frame=base_link, an obstacle at the robot's
-         physical front showed up BEHIND the model in the LaserScan display -
-         i.e. scan angle 0 pointed backward. Without this 180 deg yaw, every
-         scan was projected into base_link mirrored front-to-back, so
-         slam_toolbox built a map whose content (walls) was correct in shape
-         but rotated 180 deg from true room layout relative to the
-         (correctly-tracked, wheel+gyro) robot pose - the "forward drives
-         backward on the map" symptom. Wheel odometry / EKF heading were
-         independently verified correct (rotation-sense test) before landing
-         on this fix, so no other code changes were needed. -->
-    <origin xyz="0.0 0.0 0.170" rpy="0 0 ${pi}"/>
+    <!-- RPLIDAR C1 yaw offset from base_link +X to the lidar scan-zero.
+         pi = zero faces the chassis REAR (verified on the reference robot
+         2026-07-13 and on qb3rt-7 2026-07-19: a door at the physical nose
+         reads at raw scan angle ~180 deg, so +pi maps it to base +X).
+         If a unit's lidar is mounted with zero facing FRONT, pass
+         lidar_yaw:=0. NOTE (qb3rt-7, 2026-07-19): this unit ALSO needed
+         drive_inverted:=true in wave_rover_bridge.yaml (+x rolled toward the
+         physical rear) - the drive and scan conventions are independent
+         hardware quirks, verify both on each unit before fleet rollout. -->
+    <origin xyz="0.0 0.0 0.170" rpy="0 0 $(arg lidar_yaw)"/>
   </joint>
 </robot>
